Commit message: Docs & Update: Modify README and fine-tune nav params

File: src/gazebo_modele/urdf/model.urdf (robot description, URDF)
Before this commit: robot lio, 9 links, 8 joints
Links:
- added link camera_link, mass 0.05; collision box size=0.02 0.04 0.03; visual box size=0.02 0.04 0.03
Joints:
- added joint camera_joint: type fixed, parent base_link, child camera_link, origin xyz=0.12 0 0.08 rpy=0 0 0
